Commit message: Update Fanuc M900iB Package

File: fanuc_m900ib_support/urdf/m900ib_macro.xacro (robot description, xacro)
@@ -176,5 +176,5 @@
     <link name="${prefix}base" />
     <joint name="${prefix}base_link-base" type="fixed">
-      <origin xyz="0 0 0.450" rpy="0 0 0"/>
+      <origin xyz="0 0 0.950" rpy="0 0 0"/>
       <parent link="${prefix}base_link"/>
       <child link="${prefix}base"/>

Commit message: Update tool mesh and .xacro file

File: fanuc_m900ib_support/urdf/m900ib_macro.xacro (robot description, xacro)
@@ -24,5 +24,5 @@
         <origin xyz="0 0 0.601" rpy="0 0 0"/>
         <geometry>
-          <mesh filename="package://fanuc_m900ib_support/meshes/m900ib/visual/link_1.stl"/>
+          <mesh filename="package://fanuc_m900ib_support/meshes/m900ib/visual/link_1.dae"/>
         </geometry>
         <xacro:material_fanuc_yellow />
@@ -39,5 +39,5 @@
         <origin xyz="0 0 0" rpy="0 0 3.14159265359"/>
         <geometry>
-          <mesh filename="package://fanuc_m900ib_support/meshes/m900ib/visual/link_2.stl"/>
+          <mesh filename="package://fanuc_m900ib_support/meshes/m900ib/visual/link_2.dae"/>
         </geometry>
         <xacro:material_fanuc_yellow />
@@ -54,5 +54,5 @@
         <origin xyz="0 0 0" rpy="0 0 0"/>
         <geometry>
-          <mesh filename="package://fanuc_m900ib_support/meshes/m900ib/visual/link_3.stl"/>
+          <mesh filename="package://fanuc_m900ib_support/meshes/m900ib/visual/link_3.dae"/>
         </geometry>
         <xacro:material_fanuc_yellow />
@@ -114,5 +114,5 @@
         <origin xyz="-0.32955 -0.07795 -0.02692" rpy="0 0 ${-m_pi_2}"/>
         <geometry>
-          <mesh filename="package://fanuc_m900ib_support/meshes/m900ib/visual/fsw.stl"/>
+          <mesh filename="package://fanuc_m900ib_support/meshes/m900ib/visual/fsw.dae"/>
         </geometry>
         <xacro:material_fanuc_grey />
@@ -176,5 +176,5 @@
     <link name="${prefix}base" />
     <joint name="${prefix}base_link-base" type="fixed">
-      <origin xyz="0 0 0.950" rpy="0 0 0"/>
+      <origin xyz="0 0 0.940" rpy="0 0 0"/>
       <parent link="${prefix}base_link"/>
       <child link="${prefix}base"/>
